Commit message: fix(sim): render the camera and cover the full operator workspace
Two world/description fixes so the camera produces useful frames:

* Launch worlds/cell.sdf (stock empty.sdf + the gz Sensors system) instead of
  the bare empty.sdf. empty.sdf never loads Sensors, so the cell camera was
  advertised but never rendered — /camera/image stayed silent and perception
  went blind (safety fail-safed to 'lost'). Headless uses --headless-rendering
  so the sensor renders offscreen via EGL.
* Raise, centre and widen the camera mast (camera_link world z 2.40 m, pitch
  1.2 rad, hfov 1.5 rad). The old low/narrow mast only framed the tray; the
  operator's standing/approach poses projected above the frame, so perception
  lost the operator between tray reaches. The new FOV covers the whole working
  volume. Spawn the operator marker at the constant marker height (z=0.95).

File: src/safecollab/urdf/cell.xacro (robot description, xacro)
@@ -84,10 +84,17 @@
   </xacro:kitting_arm>
   <!-- ================= camera sensor (Stream C) ================= -->
-  <!-- mast rising from the table to hold the camera looking down at the cell -->
-  <xacro:box_link name="camera_mast" sx="0.04" sy="0.04" sz="0.90" mass="2.0" material="cam_mat"/>
+  <!-- Mast rising from the table to hold the overhead camera. It is tall
+       (1.70 m) and the camera sits high (world z = 2.40) and centred on the
+       cell (y = 0) so the camera FOV covers the WHOLE operator working volume
+       (x 0.35..0.9, y ±0.65, z 0.82..1.10), not just the tray. With the older
+       low/narrow mast the standing/approach parts of the operator path fell
+       outside the frame, perception lost the operator between tray reaches, and
+       the safety loop dropped to the 'lost' fail-safe. See docs/VALIDATE.md and
+       perception_node.cam_to_world_transform (its defaults mirror this chain). -->
+  <xacro:box_link name="camera_mast" sx="0.04" sy="0.04" sz="1.70" mass="2.0" material="cam_mat"/>
   <joint name="top_to_mast" type="fixed">
     <parent link="table_top"/>
     <child  link="camera_mast"/>
-    <origin xyz="-0.55 0.35 0.45" rpy="0 0 0"/>
+    <origin xyz="-0.55 0.0 0.85" rpy="0 0 0"/>
   </joint>
   <link name="camera_link">
@@ -104,9 +111,11 @@
     </inertial>
   </link>
-  <!-- mount the camera at the top of the mast, pitched down to view the tray/cell -->
+  <!-- mount the camera at the top of the mast, pitched down to view the cell.
+       camera_link world pose: table_top(0,0,0.74) + top_to_mast(-0.55,0,0.85)
+       + mast_to_camera(0.10,0,0.81) = (-0.45, 0, 2.40).  pitch = 1.2 rad. -->
   <joint name="mast_to_camera" type="fixed">
     <parent link="camera_mast"/>
     <child  link="camera_link"/>
-    <origin xyz="0.10 0.0 0.45" rpy="0 1.0 0"/>
+    <origin xyz="0.10 0.0 0.81" rpy="0 1.2 0"/>
   </joint>
   <!-- optical frame: REP-103 camera optical convention (z forward, x right, y down) -->
@@ -127,5 +136,8 @@
       <topic>camera/image</topic>
       <camera>
-        <horizontal_fov>1.0472</horizontal_fov>
+        <!-- 1.5 rad (~86 deg): wide enough that the raised overhead camera
+             sees the entire operator working volume (see top_to_mast comment).
+             perception_node._CAM_HFOV mirrors this value. -->
+        <horizontal_fov>1.5</horizontal_fov>
         <image>
           <width>640</width>
