Commit message: feat(robot): UR5e + MoveIt-planned pick-and-place (retire cylinder arm)
Replace the hand-built cylinder arm and its hand-solved joint poses with a real
Universal Robots UR5e whose kitting motion is planned by MoveIt, while keeping
the ISO/TS 15066 SSM speed-scaling loop (safety_monitor → /safety/scale →
motion_node retime) completely intact — MoveIt only changes how the nominal
trajectory is generated, not how safety governs it.

Robot
- Mount the ur_description UR5e macro in cell.xacro via gz_ros2_control (the
  ur_simulation_gz ur_ros2_control wiring). UR joint names already match
  config/controllers.yaml and the motion pipeline, so arm_controller +
  joint_state_broadcaster and motion_node's /arm_controller/joint_trajectory
  path are unchanged. Add ur-description + ur-simulation-gz to the Dockerfile.
- safety.yaml robot_frames tcp/link_6/link_3 → UR tool0/wrist_3_link/forearm_link.

Planner (replaces task_node)
- planner_node uses MoveItPy + the deterministic Pilz industrial planner. Each
  Cartesian tool target is resolved ONCE to a joint config with FK-verified IK
  (KDL is the only solver packaged and is non-deterministic; seed shoulder_pan at
  the target, try both world/base_link pose frames, accept only a solution whose
  tool0 FK lands within 20 mm of the world target), cached, then reached with a
  Pilz PTP. Legs are paced to the planned trajectory duration. The dense position
  trajectory is published on /motion/nominal_trajectory, which motion_node retimes
  for SSM — so no motion_node/retime changes were needed.
- Add moveit + moveit-py + pilz + ur-moveit-config to the Dockerfile; vendor the
  MoveIt config (SRDF, kinematics, Pilz limits) under config/ and srdf/. The
  launch assembles the MoveIt params (reshaping planning_pipelines to the
  pipeline_names form MoveItCpp needs) and passes them to planner_node.

Scenario / tests
- human_node: push the standing pose clear of the arm-at-tray (unambiguous green),
  randomise the standing dwell to break the operator/arm beat-frequency lock, and
  hold the tray reach so it co-occurs with the arm at the shared tray (red).
- AT-6: extend the window (150→210 s) and lower the recurrence floor (3→2
  escalations) — the UR5e's planned motion makes the red-triggering tray
  co-occupancy rarer per unit time; ≥2 distinct-path escalations still proves the
  behaviour generalises. Replace the task_node state-machine unit tests with
  planner-plan tests.

Retire the now-dead urdf/arm.xacro and safecollab/task_node.py.

Verified in the production image (docker build with the MoveIt layer): the UR5e
does real pick-and-place (0 mm IK, tool0 to the bin/tray), AT-1..AT-5 and AT-6
pass (run individually), unit suite 285 pass at 99.8% coverage.

File: src/safecollab/urdf/cell.xacro (robot description, xacro)
@@ -8,8 +8,11 @@
        * one shared kitting tray (drop location, co-occupied with the operator)
        * a down-looking camera sensor publishing on /camera/image (for Stream C)
-       * the 6-DOF arm (from arm.xacro) mounted on the table
+       * the 6-DOF Universal Robots UR5e (ur_description macro) mounted on the table
        * the gz_ros2_control::GazeboSimROS2ControlPlugin loading controllers.yaml -->
 <robot name="safecollab_cell" xmlns:xacro="http://www.ros.org/wiki/xacro">
-  <xacro:include filename="$(find safecollab)/urdf/arm.xacro"/>
+  <!-- Universal Robots UR5e: real model + solved kinematics from ur_description;
+       ur_simulation_gz supplies the gz_ros2_control wiring (ur_ros2_control macro). -->
+  <xacro:include filename="$(find ur_description)/urdf/ur_macro.xacro"/>
+  <xacro:include filename="$(find ur_simulation_gz)/urdf/ur_gz.ros2_control.xacro"/>
   <!-- ================= materials ================= -->
   <material name="table_mat"><color rgba="0.6 0.45 0.3 1.0"/></material>
@@ -79,8 +82,24 @@
     <origin xyz="0.35 0.0 0.02" rpy="0 0 0"/>
   </joint>
-  <!-- ================= the arm (mounted on the table top, centred at the back) ================= -->
-  <xacro:kitting_arm parent="table_top">
+  <!-- ================= the arm: Universal Robots UR5e ================= -->
+  <!-- Mounted on the table top toward the back. UR joint names already match
+       config/controllers.yaml, so the arm_controller + joint_state_broadcaster
+       wiring is unchanged. force_abs_paths=true so gz (and RViz) resolve the UR
+       meshes by absolute path. The gz_ros2_control PLUGIN is declared once below
+       (shared with nothing else); ur_ros2_control adds the <ros2_control> system
+       block with position/velocity/effort interfaces on the six joints. -->
+  <xacro:property name="ur_cfg" value="$(find ur_description)/config/ur5e"/>
+  <xacro:ur_robot
+      name="ur5e"
+      tf_prefix=""
+      parent="table_top"
+      joint_limits_parameters_file="${ur_cfg}/joint_limits.yaml"
+      kinematics_parameters_file="${ur_cfg}/default_kinematics.yaml"
+      physical_parameters_file="${ur_cfg}/physical_parameters.yaml"
+      visual_parameters_file="${ur_cfg}/visual_parameters.yaml"
+      force_abs_paths="true">
     <origin xyz="-0.10 0.0 0.0" rpy="0 0 0"/>
-  </xacro:kitting_arm>
+  </xacro:ur_robot>
+  <xacro:ur_ros2_control name="ur5e" tf_prefix=""/>
   <!-- ================= camera sensor (Stream C) ================= -->
   <!-- Mast rising from the table to hold the overhead camera. It is tall

Commit message: fix(demo): make the UR5e kitting demo actually run its task under SSM
The UR5e + MoveIt swap looked broken in the live demo: the arm jerked and
barely moved, the operator was never green, one feeder bin was unreachable,
and picks near the operator were abandoned half-way. Four independent causes:

- motion_node: /joint_states is published in the broadcaster's alphabetical
  order (elbow, shoulder_lift, shoulder_pan, ...) but the Pilz trajectory uses
  ur_manipulator group order (shoulder_pan first). The resume/hold waypoint was
  spliced with shoulder_pan <-> elbow swapped, scrambling the command. Realign
  the current state by joint name before use.

- perception_node: detection confidence was the blob's fraction of the whole
  frame (~0.02 for the overhead marker), which maxed the sigma term and inflated
  the ISO/TS 15066 thresholds (d_yellow ~ 1.0 m, larger than the cell) so the
  operator never registered green. Confidence now scores the blob against an
  expected operator size; a clean detection is confident (sigma ~ 0.10 m) and the
  robot gets a real full-speed window.

- cell.xacro: feeder bins sat on the shoulder-singularity line (base-rel x ~ 0),
  where the UR5e's lateral shoulder offset made the mirrored +y reach unreachable.
  Move both bins forward-of-centre to (0.15, +/-0.35) on a slightly widened table
  for a well-conditioned front-side pick.

- planner_node: legs advanced by wall-clock time, so an SSM slow-down/stop near
  the operator abandoned the in-progress pick. Pace closed-loop: wait until the
  arm reaches each leg goal (name-aligned joint check, generous timeout) before
  advancing, so a stop only delays the pick and the arm completes it when clear.

Verified headless in perceived mode: both bins reach 0 mm, the SSM zone cycles
green/yellow/red, and the task flows through every leg. Unit suite 288 pass.

File: src/safecollab/urdf/cell.xacro (robot description, xacro)
@@ -42,5 +42,11 @@
   <xacro:property name="table_h"  value="0.74"/>   <!-- table top height above floor -->
   <xacro:property name="table_sx" value="1.20"/>
-  <xacro:property name="table_sy" value="0.80"/>
+  <!-- table depth (y): widened from 0.80 so the two feeder bins sit on the
+       robot's LEFT/RIGHT flanks at a natural UR5e reach radius (~0.41 m from
+       the base) instead of tucked in behind/under the base. The old bins at
+       base-rel (-0.20, ±0.25) forced a folded back-over-the-shoulder reach —
+       the arm looked like it "stopped short" of the box. Side bins give a clean
+       elbow-up side pick and keep bin work lateral (clear of the front operator). -->
+  <xacro:property name="table_sy" value="1.05"/>
   <!-- ================= world ================= -->
   <link name="world"/>
@@ -62,9 +68,17 @@
   </joint>
   <!-- ================= feeder bins (pick) ================= -->
+  <!-- Bins flank the base FORWARD-of-centre at world (0.15, ±0.35):
+       base-rel (0.25, ±0.35), radius ≈ 0.43 m. The forward offset is key:
+       bins on the pure-side line (base-rel x ≈ 0) sit near the UR5e SHOULDER
+       SINGULARITY (wrist centre over the shoulder axis), where the +y reach
+       becomes an awkward near-singular config the arm can't cleanly complete —
+       so one bin was reachable and the mirrored one was not. Pushing the bins
+       forward moves both off that singular line into a well-conditioned
+       front-side reach. planner_node's bin targets mirror these coordinates. -->
   <xacro:box_link name="bin_left"  sx="0.15" sy="0.15" sz="0.08" mass="0.5" material="bin_mat"/>
   <joint name="top_to_bin_left" type="fixed">
     <parent link="table_top"/>
     <child  link="bin_left"/>
-    <origin xyz="-0.30 0.25 0.04" rpy="0 0 0"/>
+    <origin xyz="0.15 0.35 0.04" rpy="0 0 0"/>
   </joint>
   <xacro:box_link name="bin_right" sx="0.15" sy="0.15" sz="0.08" mass="0.5" material="bin_mat"/>
@@ -72,5 +86,5 @@
     <parent link="table_top"/>
     <child  link="bin_right"/>
-    <origin xyz="-0.30 -0.25 0.04" rpy="0 0 0"/>
+    <origin xyz="0.15 -0.35 0.04" rpy="0 0 0"/>
   </joint>
   <!-- ================= shared kitting tray (drop) ================= -->
