Commit message: fix(arm): re-proportion links and re-solve poses to stop the arm folding
The arm reached the pick/drop targets correctly, but the intermediate links
folded over themselves: with a 0.40 + 0.35 m upper-arm/forearm and a 0.28 m
wrist, reaching targets only ~0.32-0.46 m away at near-shoulder height forced
the elbow ~0.45 m above the shoulder and the forearm to double back over the
upper arm (the "folds in itself" posture), operating near a folded elbow
singularity throughout. home also pointed the arm straight up (tcp at z≈1.79).

Cause is geometric, not an IK error: the links were far longer than the reach.
Fix: proportion the arm to the cell — upper arm/forearm 0.25 m each and a SHORT
wrist (0.06+0.05+0.05 = 0.16 m) so the tool sits just above the target when
pointing down instead of forcing the whole arm up-and-over. The seven _Q poses
are re-solved with a closed-form planar 2R IK (elbow-up branch, tool pointing
straight down) against the new chain. Verified per pose: 0 mm TCP error, all
joints within [-π, π], and from the elbow the chain descends monotonically in
BOTH height and radius to the target — a clean inverted-V reach, no fold. The
TCP targets are unchanged (pick/drop z≈0.80 m, hover z≈0.95 m) so the safety
min-distance behaviour is identical; home is now a compact hover over the work
area. robot_state_publisher parses the new xacro and AT-1..AT-5 / AT-6 pass.

File: src/safecollab/urdf/arm.xacro (robot description, xacro)
@@ -39,12 +39,21 @@
        *origin: placement of base_link wrt parent -->
   <xacro:macro name="kitting_arm" params="parent *origin">
-    <!-- link lengths (m) -->
+    <!-- link lengths (m).
+         Proportioned to the cell: the pick/drop targets sit only ~0.32-0.46 m
+         from the shoulder at roughly shoulder height, so the upper arm + forearm
+         (l_2 + l_3) are kept short enough that reaching them needs only a modest
+         elbow bend (~100 deg at the bins) instead of folding the forearm back
+         over the upper arm. The wrist (l_4 + l_5 + l_6) is deliberately SHORT so
+         the tool sits just above the target when pointing straight down, rather
+         than forcing the whole arm up-and-over (which produced the earlier
+         "folds in itself" posture). Poses in task_node._Q are IK-solved for this
+         chain (elbow-up, tool-down); changing a length here means re-solving them. -->
     <xacro:property name="l_base"  value="0.10"/>
     <xacro:property name="l_1"     value="0.15"/>
-    <xacro:property name="l_2"     value="0.40"/>
-    <xacro:property name="l_3"     value="0.35"/>
-    <xacro:property name="l_4"     value="0.10"/>
-    <xacro:property name="l_5"     value="0.10"/>
-    <xacro:property name="l_6"     value="0.08"/>
+    <xacro:property name="l_2"     value="0.25"/>
+    <xacro:property name="l_3"     value="0.25"/>
+    <xacro:property name="l_4"     value="0.06"/>
+    <xacro:property name="l_5"     value="0.05"/>
+    <xacro:property name="l_6"     value="0.05"/>
     <!-- common revolute limits -->
     <xacro:property name="j_eff"   value="100.0"/>
